File: sparrow.sch (EAGLE design)
At the start: 192 parts, among them IC1 LAN8720AVIAS, IC2 TLV320AIC3100VIAS, IC3 TPS2500, IC4 SKYWORKS_AAT4280ASC70JW-8-NOT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, IC5 SKYWORKS_AAT4280ASC70JW-8-NOT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, IC6 SKYWORKS_AAT4280ASC70JW-8-NOT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, IC7 SKYWORKS_AAT4280ASC70JW-8-NOT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, IC8 SKYWORKS_AAT4280ASC70JW-8-NOT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, IC9 FXMA10820-DFN, X1 ABS07-32768, X2 12MHz, X3 32.768KHz, X4 50MHZ, Y2 16MHz

Commit message: power routing, added LEDs, several last-minute improvements
Parts:
- removed C70: 2.2p, anykey:CAP_CERAMIC0402
- removed C71, C73: 1p, anykey:CAP_CERAMIC0402
- removed L10: 3.3nH, anykey:INDUCTOR0402
- removed L8: 4.7nH, anykey:INDUCTOR0402
- removed L9: 10nH, anykey:INDUCTOR0402
- added BAL1: BALUNWLCSP, anykey:BALUNWLCSP
- added LED2, LED3, LED4: (no value), anykey:LED0603
- added R40, R41: 33, anykey:R-EU_0603
- added R42: 10K, anykey:R-EU_0603
- added R43, R44, R45: 806, anykey:R-EU_0603
- 5VDC_IN: value (none) -> 2A max
- ANT1, ANT2: value (none) -> 2.4GHz 50Ω
- BATT: value (none) -> BATTERY_WITH_HOLDER; device anykey:HEADER-1X2JST-PH-H -> anykey:BATTERY_WITH_HOLDER
- C1: value 1000p -> 1n
- C10, C8, C9: value 4.7u -> 4µ7
- C12, C13, C14, C15, C16, C17, C18, C19, C20, C21, C24, C25, C26, C3, C30, C31, C32, C33, C34, C35, C36, C37, C38, C39, C4, C43, C45, C47, C49, C5, C58, C6, C62, C63, C64, C7, C74, C75: value 0.1µ -> 100n
- C52, C53: value (none) -> 1µ
- C54: value (none) -> 100n
- C55: value (none) -> 2p2
- C61: value 0.047µ -> 47n
- C72: value 2.2p -> 2n2
- D1, D2, D3, D4, D5: value (none) -> MBR230LSFT1
- HP: value (none) -> HP
- I2C0: value (none) -> I2C0
- I2C1: value (none) -> I2C1
- L1: value 10µH -> 10µ
- L5: value (none) -> 2n2
- L6: value (none) -> DNP
- L7: value 2.2µ -> 2µ2
- LIM: value JUMPERSOLDER_CLOSED -> JUMPERSOLDER_OPEN; device anykey:JUMPERSOLDER_CLOSED -> anykey:JUMPERSOLDER_OPEN
- LINE: value (none) -> LINE
- LS: value (none) -> LS
- MIC: value (none) -> MIC
- R2: value 2.4M -> 2M4
- R21: value (none) -> 2K2
- R29, R34: value (none) -> 100K
- SD_CARD: value SD_CARD -> SD_CARDEXTENDED; device anykey:SD_CARD -> anykey:SD_CARDEXTENDED
- UART2: value (none) -> UART2
- UART_5V: value (none) -> UART_5V
- X3: value 32.768KHz -> 32768
- renumbered U$6 to ETH, Y2 to X5
Connections:
- net N$19 renamed ETH_LED1_CURR
- net N$20 renamed VUSB1_V5_OUT
- net N$22 renamed ETH_LED2_CURR
- net N$9 renamed CHARGE_!CHRG_CURR
- removed net AVAIL1: MCU.P3_1
- removed net BT_ANT_UNBAL: C70.P$2, C71.P$2, L10.1
- removed net ETH_RTERM: C33.P$1, R19.2, R20.1
- removed net ETH_TTERM: C32.P$1, R17.2, R18.1
- new net ETH_!INT: IC1.!INT!/REFCLK0, MCU.P3_1, R42.1
- new net ETH_REF_CLK_MAC: MCU.CLK0, R40.1
- new net ETH_REF_CLK_PHY: IC1.XTAL1/CLKIN, R41.2
- new net N$1: LED2.ANODE, R45.2
- new net N$2: LED3.ANODE, R43.2
- new net N$3: LED4.ANODE, R44.2
- net AVAIL7: now also R45.1
- net AVAIL8: now also R43.1
- net AVAIL9: now also R44.1
- net BT_ANT: now also BAL1.UNBAL; no longer C73.P$2, L10.2
- net BT_ANT1: now also BAL1.BAL2; no longer L8.1, L9.2
- net BT_ANT2: now also BAL1.BAL1; no longer C70.P$1, L8.2
- net BT_VDD_PA: now also BAL1.DC; no longer L9.1
- net BT_XC1: now also C67.P$1, X5.1; no longer C66.P$1, X5.2
- net BT_XC2: now also C66.P$1, X5.2; no longer C67.P$1, X5.1
- net ETH_REF_CLK: now also R40.2, R41.1; no longer IC1.XTAL1/CLKIN, MCU.CLK0
- net GND: now also BAL1.GND, BATT.-, BATT.HOLDER, LED2.CATHODE, LED3.CATHODE, LED4.CATHODE, MCU1.VSS; no longer BATT.2, C71.P$1, C73.P$1
- net VBAT: now also BATT.+; no longer BATT.1
- net VETH33: now also C32.P$1, C33.P$1, R17.2, R18.1, R19.2, R20.1, R42.2
Other:
- note added: "Note: Bulk in and out caps (C57, C59, C60) should be connected to PGND, not GND to prevent excessive switching noise on common GND. Only one star connection from PGND to GND below TPS2500."
- note added: "Note: R34 only needed for first revision of NRF51822. DNP for Rev. 2 and up."
- note added: "PGND"
- note added: "Place series terminations close to clock, keep both lines same length"
- moved on the sheet: ANT2, C1, C31, C32, C33, C38, C39, C40, C41, C42, C43, C44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
