File: sparrow.sch (EAGLE design)
At the start: 196 parts, among them IC1 LAN8720AVIAS, IC2 TLV320AIC3100VIAS, IC3 TPS2500, IC4 SKYWORKS_AAT4280ASC70JW-8-NOT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, IC5 SKYWORKS_AAT4280ASC70JW-8-NOT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, IC6 SKYWORKS_AAT4280ASC70JW-8-NOT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, IC7 SKYWORKS_AAT4280ASC70JW-8-NOT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, IC8 SKYWORKS_AAT4280ASC70JW-8-NOT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, IC9 FXMA10820-DFN, X1 ABS07-32768, X2 12MHz, X3 32768, X4 50MHZ, X5 16MHz

Commit message: RC1
Parts:
- added HEADPHONE: AUDIOJACK-STEREO-3PCUI_SJ_3523, anykey:AUDIOJACK-STEREO-3PCUI_SJ_3523
- I2S: value HEADER-1X10ROUND -> HEADER-2X5SMD-1.27MM; device anykey:HEADER-1X10ROUND -> anykey:HEADER-2X5SMD-1.27MM
Connections:
- net MIC renamed N$4
- net GND: now also HEADPHONE.SLEEVE
- net HP_L: now also HEADPHONE.TIP
- net HP_R: now also HEADPHONE.RING
- net I2S_RX_MCLK: now also I2S.9; no longer I2S.3
- net I2S_RX_SCK: now also I2S.3; no longer I2S.4
- net I2S_RX_SD: now also I2S.7; no longer I2S.8
- net I2S_RX_WS: now also I2S.5; no longer I2S.6
- net I2S_TX_SCK: now also I2S.4; no longer I2S.5
- net I2S_TX_SD: now also I2S.8; no longer I2S.9
- net I2S_TX_WS: now also I2S.6; no longer I2S.7
Changed lines of the file:
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@@
 <part name="RX_SCK" library="anykey" deviceset="JUMPER" device="SOLDER_CLOSED"/>
 <part name="MCLK" library="anykey" deviceset="JUMPER" device="SOLDER_CLOSED"/>
-<part name="I2S" library="anykey" deviceset="HEADER-1X10" device="ROUND" value="HEADER-1X10ROUND"/>
 <part name="U$48" library="anykey" deviceset="VD33" device=""/>
 <part name="U$49" library="anykey" deviceset="GND" device=""/>
@@
 <part name="LED4" library="anykey" deviceset="LED" device="0603"/>
 <part name="U$19" library="anykey" deviceset="GND" device=""/>
+<part name="I2S" library="anykey" deviceset="HEADER-2X5" device="SMD-1.27MM"/>
+<part name="HEADPHONE" library="anykey" deviceset="AUDIOJACK-STEREO-3P" device="CUI_SJ_3523"/>
 </parts>
 <sheets>
@@
 <instance part="RX_SCK" gate="G$1" x="2.54" y="25.4"/>
 <instance part="MCLK" gate="G$1" x="2.54" y="22.86"/>
-<instance part="I2S" gate="G$1" x="-10.16" y="10.16" rot="R270"/>
 <instance part="U$48" gate="G$1" x="7.62" y="15.24"/>
 <instance part="U$49" gate="G$1" x="7.62" y="7.62"/>
 <instance part="A_SDA" gate="G$1" x="2.54" y="43.18"/>
 <instance part="A_SCL" gate="G$1" x="2.54" y="45.72"/>
+<instance part="I2S" gate="G$1" x="-12.7" y="-7.62" rot="R270"/>
+<instance part="HEADPHONE" gate="G$1" x="139.7" y="25.4"/>
 </instances>
 <busses>
@@
 <wire x1="116.84" y1="25.4" x2="91.44" y2="25.4" width="0.1524" layer="91"/>
 <junction x="91.44" y="25.4"/>
+<wire x1="127" y1="17.78" x2="91.44" y2="17.78" width="0.1524" layer="91"/>
+<junction x="91.44" y="17.78"/>
+<wire x1="127" y1="17.78" x2="127" y2="22.86" width="0.1524" layer="91"/>
+<pinref part="HEADPHONE" gate="G$1" pin="SLEEVE"/>
+<wire x1="127" y1="22.86" x2="129.54" y2="22.86" width="0.1524" layer="91"/>
 </segment>
 <segment>
@@
 <pinref part="U$49" gate="G$1" pin="GND"/>
 <wire x1="7.62" y1="7.62" x2="7.62" y2="12.7" width="0.1524" layer="91"/>
+<wire x1="7.62" y1="12.7" x2="-5.08" y2="12.7" width="0.1524" layer="91"/>
 <pinref part="I2S" gate="G$1" pin="2"/>
-<wire x1="7.62" y1="12.7" x2="-2.54" y2="12.7" width="0.1524" layer="91"/>
-<wire x1="-2.54" y1="12.7" x2="-2.54" y2="10.16" width="0.1524" layer="91"/>
+<wire x1="-5.08" y1="12.7" x2="-5.08" y2="-7.62" width="0.1524" layer="91"/>
 </segment>
 </net>
@@
 <pinref part="HP" gate="A" pin="1"/>
 <wire x1="109.22" y1="27.94" x2="116.84" y2="27.94" width="0.1524" layer="91"/>
+<pinref part="HEADPHONE" gate="G$1" pin="TIP"/>
+<wire x1="116.84" y1="27.94" x2="129.54" y2="27.94" width="0.1524" layer="91"/>
+<junction x="116.84" y="27.94"/>
 </segment>
 </net>
@@
 <pinref part="HP" gate="A" pin="3"/>
 <wire x1="109.22" y1="22.86" x2="116.84" y2="22.86" width="0.1524" layer="91"/>
+<wire x1="116.84" y1="22.86" x2="124.46" y2="22.86" width="0.1524" layer="91"/>
+<junction x="116.84" y="22.86"/>
+<wire x1="124.46" y1="22.86" x2="124.46" y2="25.4" width="0.1524" layer="91"/>
+<pinref part="HEADPHONE" gate="G$1" pin="RING"/>
+<wire x1="124.46" y1="25.4" x2="129.54" y2="25.4" width="0.1524" layer="91"/>
 </segment>
 </net>
@@
 </segment>
 </net>
-<net name="MIC" class="0">
-<segment>
-<pinref part="C54" gate="G$1" pin="P$1"/>
-<wire x1="43.18" y1="66.04" x2="40.64" y2="66.04" width="0.1524" layer="91"/>
-<pinref part="R21" gate="G$1" pin="1"/>
-<wire x1="40.64" y1="66.04" x2="40.64" y2="63.5" width="0.1524" layer="91"/>
-<wire x1="40.64" y1="63.5" x2="40.64" y2="58.42" width="0.1524" layer="91"/>
-<junction x="40.64" y="63.5"/>
-<pinref part="IC2" gate="G$1" pin="VOL/MICDET"/>
-<wire x1="40.64" y1="58.42" x2="55.88" y2="58.42" width="0.1524" layer="91"/>
-<pinref part="MIC" gate="G$1" pin="2"/>
-<wire x1="33.02" y1="66.04" x2="40.64" y2="66.04" width="0.1524" layer="91"/>
-<junction x="40.64" y="66.04"/>
-</segment>
-</net>
 <net name="AUDIO_!RESET" class="0">
 <segment>
@@
 <wire x1="-2.54" y1="38.1" x2="-20.32" y2="38.1" width="0.1524" layer="91"/>
 <label x="-40.64" y="38.1" size="1.778" layer="95"/>
-<pinref part="I2S" gate="G$1" pin="9"/>
 <wire x1="-20.32" y1="38.1" x2="-43.18" y2="38.1" width="0.1524" layer="91"/>
-<wire x1="-20.32" y1="10.16" x2="-20.32" y2="38.1" width="0.1524" layer="91"/>
+<wire x1="-20.32" y1="-7.62" x2="-20.32" y2="38.1" width="0.1524" layer="91"/>
 <junction x="-20.32" y="38.1"/>
+<pinref part="I2S" gate="G$1" pin="8"/>
 </segment>
 </net>
@@
 <wire x1="-2.54" y1="35.56" x2="-17.78" y2="35.56" width="0.1524" layer="91"/>
 <label x="-40.64" y="35.56" size="1.778" layer="95"/>
-<pinref part="I2S" gate="G$1" pin="8"/>
 <wire x1="-17.78" y1="35.56" x2="-43.18" y2="35.56" width="0.1524" layer="91"/>
-<wire x1="-17.78" y1="10.16" x2="-17.78" y2="35.56" width="0.1524" layer="91"/>
+<wire x1="-17.78" y1="-7.62" x2="-17.78" y2="35.56" width="0.1524" layer="91"/>
 <junction x="-17.78" y="35.56"/>
+<pinref part="I2S" gate="G$1" pin="7"/>
 </segment>
 </net>
 <net name="I2S_TX_WS" class="0">
 <segment>
-<pinref part="I2S" gate="G$1" pin="7"/>
 <pinref part="TX_WS" gate="G$1" pin="P$1"/>
 <wire x1="-2.54" y1="33.02" x2="-15.24" y2="33.02" width="0.1524" layer="91"/>
 <label x="-40.64" y="33.02" size="1.778" layer="95"/>
 <wire x1="-15.24" y1="33.02" x2="-43.18" y2="33.02" width="0.1524" layer="91"/>
-<wire x1="-15.24" y1="10.16" x2="-15.24" y2="33.02" width="0.1524" layer="91"/>
+<wire x1="-15.24" y1="-7.62" x2="-15.24" y2="33.02" width="0.1524" layer="91"/>
 <junction x="-15.24" y="33.02"/>
+<pinref part="I2S" gate="G$1" pin="6"/>
 </segment>
 </net>
 <net name="I2S_RX_WS" class="0">
 <segment>
-<pinref part="I2S" gate="G$1" pin="6"/>
 <pinref part="RX_WS" gate="G$1" pin="P$1"/>
 <wire x1="-2.54" y1="30.48" x2="-12.7" y2="30.48" width="0.1524" layer="91"/>
 <label x="-40.64" y="30.48" size="1.778" layer="95"/>
 <wire x1="-12.7" y1="30.48" x2="-43.18" y2="30.48" width="0.1524" layer="91"/>
-<wire x1="-12.7" y1="10.16" x2="-12.7" y2="30.48" width="0.1524" layer="91"/>
+<wire x1="-12.7" y1="-7.62" x2="-12.7" y2="30.48" width="0.1524" layer="91"/>
 <junction x="-12.7" y="30.48"/>
+<pinref part="I2S" gate="G$1" pin="5"/>
 </segment>
 </net>
 <net name="I2S_TX_SCK" class="0">
 <segment>
-<pinref part="I2S" gate="G$1" pin="5"/>
 <pinref part="TX_SCK" gate="G$1" pin="P$1"/>
 <wire x1="-2.54" y1="27.94" x2="-10.16" y2="27.94" width="0.1524" layer="91"/>
 <label x="-40.64" y="27.94" size="1.778" layer="95"/>
 <wire x1="-10.16" y1="27.94" x2="-43.18" y2="27.94" width="0.1524" layer="91"/>
-<wire x1="-10.16" y1="10.16" x2="-10.16" y2="27.94" width="0.1524" layer="91"/>
+<wire x1="-10.16" y1="-7.62" x2="-10.16" y2="27.94" width="0.1524" layer="91"/>
 <junction x="-10.16" y="27.94"/>
+<pinref part="I2S" gate="G$1" pin="4"/>
 </segment>
 </net>
 <net name="I2S_RX_SCK" class="0">
 <segment>
-<pinref part="I2S" gate="G$1" pin="4"/>
 <pinref part="RX_SCK" gate="G$1" pin="P$1"/>
 <wire x1="-2.54" y1="25.4" x2="-7.62" y2="25.4" width="0.1524" layer="91"/>
 <label x="-40.64" y="25.4" size="1.778" layer="95"/>
 <wire x1="-7.62" y1="25.4" x2="-43.18" y2="25.4" width="0.1524" layer="91"/>
-<wire x1="-7.62" y1="10.16" x2="-7.62" y2="25.4" width="0.1524" layer="91"/>
+<wire x1="-7.62" y1="-7.62" x2="-7.62" y2="25.4" width="0.1524" layer="91"/>
 <junction x="-7.62" y="25.4"/>
+<pinref part="I2S" gate="G$1" pin="3"/>
 </segment>
 </net>
 <net name="I2S_RX_MCLK" class="0">
 <segment>
-<pinref part="I2S" gate="G$1" pin="3"/>
 <pinref part="MCLK" gate="G$1" pin="P$1"/>
-<wire x1="-2.54" y1="22.86" x2="-5.08" y2="22.86" width="0.1524" layer="91"/>
+<wire x1="-2.54" y1="22.86" x2="-22.86" y2="22.86" width="0.1524" layer="91"/>
 <label x="-40.64" y="22.86" size="1.778" layer="95"/>
-<wire x1="-5.08" y1="22.86" x2="-43.18" y2="22.86" width="0.1524" layer="91"/>
-<wire x1="-5.08" y1="10.16" x2="-5.08" y2="22.86" width="0.1524" layer="91"/>
-<junction x="-5.08" y="22.86"/>
+<wire x1="-22.86" y1="22.86" x2="-43.18" y2="22.86" width="0.1524" layer="91"/>
+<wire x1="-22.86" y1="-7.62" x2="-22.86" y2="22.86" width="0.1524" layer="91"/>
+<junction x="-22.86" y="22.86"/>
+<pinref part="I2S" gate="G$1" pin="9"/>
 </segment>
 </net>
@@
 <net name="I2S_TX_MCLK" class="0">
 <segment>
-<pinref part="I2S" gate="G$1" pin="10"/>
-<wire x1="-43.18" y1="20.32" x2="-22.86" y2="20.32" width="0.1524" layer="91"/>
-<wire x1="-22.86" y1="20.32" x2="-22.86" y2="10.16" width="0.1524" layer="91"/>
+<wire x1="-43.18" y1="20.32" x2="-25.4" y2="20.32" width="0.1524" layer="91"/>
 <label x="-40.64" y="20.32" size="1.778" layer="95"/>
+<pinref part="I2S" gate="G$1" pin="10"/>
+<wire x1="-25.4" y1="20.32" x2="-25.4" y2="-7.62" width="0.1524" layer="91"/>
 </segment>
 </net>
@@
 <segment>
 <pinref part="U$48" gate="G$1" pin="VD33"/>
+<wire x1="7.62" y1="15.24" x2="-2.54" y2="15.24" width="0.1524" layer="91"/>
 <pinref part="I2S" gate="G$1" pin="1"/>
-<wire x1="7.62" y1="15.24" x2="0" y2="15.24" width="0.1524" layer="91"/>
-<wire x1="0" y1="15.24" x2="0" y2="10.16" width="0.1524" layer="91"/>
+<wire x1="-2.54" y1="15.24" x2="-2.54" y2="-7.62" width="0.1524" layer="91"/>
 </segment>
 </net>
@@
 </segment>
 </net>
+<net name="N$4" class="0">
+<segment>
+<pinref part="IC2" gate="G$1" pin="VOL/MICDET"/>
+<wire x1="40.64" y1="58.42" x2="55.88" y2="58.42" width="0.1524" layer="91"/>
+<pinref part="R21" gate="G$1" pin="1"/>
+<wire x1="40.64" y1="63.5" x2="40.64" y2="58.42" width="0.1524" layer="91"/>
+<junction x="40.64" y="63.5"/>
+<pinref part="C54" gate="G$1" pin="P$1"/>
+<wire x1="43.18" y1="66.04" x2="40.64" y2="66.04" width="0.1524" layer="91"/>
+<wire x1="40.64" y1="66.04" x2="40.64" y2="63.5" width="0.1524" layer="91"/>
+<junction x="40.64" y="66.04"/>
+<pinref part="MIC" gate="G$1" pin="2"/>
+<wire x1="33.02" y1="66.04" x2="40.64" y2="66.04" width="0.1524" layer="91"/>
+</segment>
+</net>

Commit message: renamed library everykey
Parts:
- !PGM, RESET: device anykey:PUSHBUTTONKMR2XX -> everykey:PUSHBUTTONKMR2XX
- 5VDC_IN: device anykey:JACK-PLUGCUI_PJ102BH -> everykey:JACK-PLUGCUI_PJ102BH
- ADC, GPIO_5V, SPI0, UART3: device anykey:HEADER-1X7ROUND -> everykey:HEADER-1X7ROUND
- ANT1, ANT2: device anykey:ANTENNA_MONOPOLE1206 -> everykey:ANTENNA_MONOPOLE1206
- A_SCL, A_SDA, MCLK, RX_SCK, RX_SD, RX_WS, SCL, SDA, TX_SCK, TX_SD, TX_WS, WL_EN: device anykey:JUMPERSOLDER_CLOSED -> everykey:JUMPERSOLDER_CLOSED
- BAL1: device anykey:BALUNWLCSP -> everykey:BALUNWLCSP
- BATT: device anykey:BATTERY_WITH_HOLDER -> everykey:BATTERY_WITH_HOLDER
- C1, C55, C61, C62, C63, C64, C66, C67, C68, C69, C72: device anykey:CAP_CERAMIC0402 -> everykey:CAP_CERAMIC0402
- C10, C11, C12, C13, C14, C15, C16, C17, C18, C19, C2, C20, C21, C22, C23, C24, C25, C26, C27, C28, C29, C3, C30, C31, C32, C33, C34, C35, C36, C37, C38, C39, C4, C40, C41, C42, C43, C44, C45, C46, C47, C48, C49, C5, C52, C53, C54, C56, C58, C6, C65, C7, C74, C75, C76, C77, C78, C79, C8, C80, C9: device anykey:CAP_CERAMIC0603 -> everykey:CAP_CERAMIC0603
- C50, C51, C57, C59: device anykey:CAP_CERAMIC0805 -> everykey:CAP_CERAMIC0805
- C60: device anykey:CPOL-EU1210 -> everykey:CPOL-EU1210
- CC_DEBUG, I2S, LPC_DEBUG, NRF_DEBUG: device anykey:HEADER-2X5SMD-1.27MM -> everykey:HEADER-2X5SMD-1.27MM
- D1, D2, D3, D4, D5: device anykey:DIODESOD123FL -> everykey:DIODESOD123FL
- ETH: device anykey:ETHERNET_JACK_LEDSRB1-125BAG1A -> everykey:ETHERNET_JACK_LEDSRB1-125BAG1A
- HEADPHONE: device anykey:AUDIOJACK-STEREO-3PCUI_SJ_3523 -> everykey:AUDIOJACK-STEREO-3PCUI_SJ_3523
- HP, LINE: device anykey:HEADER-1X3ROUND -> everykey:HEADER-1X3ROUND
- I2C0, I2C1, UART_5V: device anykey:HEADER-1X5ROUND -> everykey:HEADER-1X5ROUND
- IC1: device anykey:LAN8720AVIAS -> everykey:LAN8720AVIAS
- IC2: device anykey:TLV320AIC3100VIAS -> everykey:TLV320AIC3100VIAS
- IC3: device anykey:TPS2500SON10 -> everykey:TPS2500SON10
- IC4, IC5, IC6, IC7, IC8: device anykey:SKYWORKS_AAT4280ASC70JW-8-NOTHERMALS -> everykey:SKYWORKS_AAT4280ASC70JW-8-NOTHERMALS
- IC9: device anykey:FXMA10820-DFN -> everykey:FXMA10820-DFN
- L1, L7: device anykey:INDUCTOR40X40MM -> everykey:INDUCTOR40X40MM
- L5, L6: device anykey:INDUCTOR0402 -> everykey:INDUCTOR0402
- LED1, LED2, LED3, LED4: device anykey:LED0603 -> everykey:LED0603
- LIM: device anykey:JUMPERSOLDER_OPEN -> everykey:JUMPERSOLDER_OPEN
- LOGO2, LOGO3, LOGO4: device anykey:LOGOKRONE -> everykey:LOGOKRONE
- LS, MIC: device anykey:HEADER-1X2ROUND -> everykey:HEADER-1X2ROUND
- MCU: device anykey:LPC1837JBD144 -> everykey:LPC1837JBD144
- MCU1: device anykey:NRF51822QFN48 -> everykey:NRF51822QFN48
- PWR1: device anykey:LTC4080DFN -> everykey:LTC4080DFN
- R1, R10, R11, R12, R13, R14, R15, R16, R17, R18, R19, R2, R20, R21, R22, R23, R24, R25, R26, R27, R28, R29, R3, R30, R31, R32, R33, R34, R35, R36, R37, R38, R39, R4, R40, R41, R42, R43, R44, R45, R5, R6, R7, R8, R9: device anykey:R-EU_0603 -> everykey:R-EU_0603
- SD_CARD: device anykey:SD_CARDEXTENDED -> everykey:SD_CARDEXTENDED
- UART2: device anykey:HEADER-1X6ROUND -> everykey:HEADER-1X6ROUND
- USB0, USB1: device anykey:USB_MICROSMD -> everykey:USB_MICROSMD
- WIFI: device anykey:CC3000EXTENDED -> everykey:CC3000EXTENDED
- X1, X3: device anykey:CRYSTAL1206 -> everykey:CRYSTAL1206
- X2: device anykey:CRYSTAL_WITH_GROUNDABM8G -> everykey:CRYSTAL_WITH_GROUNDABM8G
- X4: device anykey:OSCILLATOR25X20 -> everykey:OSCILLATOR25X20
- X5: device anykey:CRYSTAL_WITH_GROUND25X20 -> everykey:CRYSTAL_WITH_GROUND25X20
