File: sparrow.sch (EAGLE design)
At the start: 201 parts, among them IC1 LAN8720AVIAS, IC2 TLV320AIC3100VIAS, IC3 TPS2500, IC4 SKYWORKS_AAT4280ASC70JW-8-NOT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, IC5 SKYWORKS_AAT4280ASC70JW-8-NOT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, IC6 SKYWORKS_AAT4280ASC70JW-8-NOT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, IC7 SKYWORKS_AAT4280ASC70JW-8-NOT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, IC8 SKYWORKS_AAT4280ASC70JW-8-NOT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, IC9 FXMA10820-DFN, X1 ABS07-32768, X2 12MHz, X3 32768, X4 50MHZ, X5 16MHz

Commit message: Last library update, DRC fixes
Parts:
- MCU: device everykey:LPC1837JBD144 -> everykey:LPC1837JBD144QFP144
Changed lines of the file:
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@@
 <part name="USB0" library="everykey" deviceset="USB_MICRO" device="SMD"/>
 <part name="U$5" library="everykey" deviceset="GND" device=""/>
-<part name="MCU" library="everykey" deviceset="LPC1837JBD144" device="" value="LPC1837"/>
+<part name="MCU" library="everykey" deviceset="LPC1837JBD144" device="QFP144" value="LPC1837"/>
 <part name="X2" library="everykey" deviceset="CRYSTAL_WITH_GROUND" device="ABM8G" value="12MHz"/>
 <part name="C65" library="everykey" deviceset="CAP_CERAMIC" device="0603" value="18p"/>

Commit message: Updated values
Parts:
- C10, C8, C9: value 4µ7 -> 4.7u
- C27, C52, C53, C56, C76, C77, C78, C79, C80: value 1µ -> 1u
- C29, C42, C44, C46, C48, L1: value 10µ -> 10u
- C40, C41: value 22µ -> 22u
- C50, C51: value 47µ -> 47u
- C55: value 2p2 -> 2.2p
- C57, C59: value 22µ 10V -> 22u 10V
- C60: value 150µ 10V -> 150u 10V
- C72, L5: value 2n2 -> 2.2n
- L7: value 2µ2 -> 2.2u
- R1: value 768k -> 768K
- R10, R11, R12, R13, R8, R9: value 12K -> 10K
- R16: value 12K1 -> 12.1K
- R17, R18, R19, R20: value 49R9 -> 49.9 1%
- R2: value 2M4 -> 2.4M
- R21, R22, R23, R38, R39: value 2K2 -> 2.2K
- R26: value 40K2 -> 40.2K
- R7: value 12K -> 12K 1%

Commit message: value tuning
Parts:
- R4, R43, R44, R45: value 806 -> 1K
Changed lines of the file:
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@@
 <part name="R2" library="everykey" deviceset="R-EU_" device="0603" value="2.4M"/>
 <part name="R3" library="everykey" deviceset="R-EU_" device="0603" value="806"/>
-<part name="R4" library="everykey" deviceset="R-EU_" device="0603" value="806"/>
+<part name="R4" library="everykey" deviceset="R-EU_" device="0603" value="1K"/>
 <part name="LED1" library="everykey" deviceset="LED" device="0603" value="CHARGE"/>
 <part name="U$3" library="everykey" deviceset="GND" device=""/>
@@
 <part name="BAL1" library="everykey" deviceset="BALUN" device="WLCSP"/>
 <part name="BATT" library="everykey" deviceset="BATTERY_WITH_HOLDER" device=""/>
-<part name="R43" library="everykey" deviceset="R-EU_" device="0603" value="806"/>
-<part name="R44" library="everykey" deviceset="R-EU_" device="0603" value="806"/>
-<part name="R45" library="everykey" deviceset="R-EU_" device="0603" value="806"/>
+<part name="R43" library="everykey" deviceset="R-EU_" device="0603" value="1K"/>
+<part name="R44" library="everykey" deviceset="R-EU_" device="0603" value="1K"/>
+<part name="R45" library="everykey" deviceset="R-EU_" device="0603" value="1K"/>
 <part name="LED2" library="everykey" deviceset="LED" device="0603"/>
 <part name="LED3" library="everykey" deviceset="LED" device="0603"/>

Commit message: Fine tuning
Parts:
- X4: value 50MHZ -> 50MHZ Silabs 501
Changed lines of the file:
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@@
 <part name="U$22" library="everykey" deviceset="VETH33" device=""/>
 <part name="U$25" library="everykey" deviceset="VETH33" device=""/>
-<part name="X4" library="everykey" deviceset="OSCILLATOR" device="25X20" value="50MHZ"/>
+<part name="X4" library="everykey" deviceset="OSCILLATOR" device="25X20" value="50MHZ Silabs 501"/>
 <part name="U$27" library="everykey" deviceset="GND" device=""/>
 <part name="C34" library="everykey" deviceset="CAP_CERAMIC" device="0603" value="100n"/>
